File: hw/main_logic_board/main_logic_board.sch (KiCad schematic (older format))
At the start: 46 parts, among them J11 SPI1, J12 UART0, J13 UART2, J14 UART4, J15 I2C1, J16 I2C2, J4 USB_A, J5 RC_OUT_1, J6 RC_OUT_2, J7 RC_OUT_3, J8 RC_OUT_4, U1 PocketBeagle, U9 USBLC6-2P6

Commit message: Finish layout
Connections:
- net 3V3_PB: no longer U1.59 (3.3V)
- no-connect marks 24 -> 25
Changed lines of the file:
@@
 $EndComp
-Wire Wire Line
-	7000 1400 7000 1350
-Wire Wire Line
-	7000 1350 7100 1350
-Connection ~ 7100 1350
-Wire Wire Line
-	7100 1350 7100 1400
 Wire Wire Line
 	7800 3700 8350 3700
@@
 Wire Wire Line
 	7350 1100 7100 1100
-Connection ~ 7100 1100
-Wire Wire Line
-	7100 1100 7100 1350
 $Comp
 L Connector:TestPoint TP3
@@
 Text Label 3500 750  2    50   ~ 0
 AIN_3V3
+Wire Wire Line
+	7000 1250 7100 1250
+Wire Wire Line
+	7100 1250 7100 1100
+Wire Wire Line
+	7000 1250 7000 1400
+Connection ~ 7100 1100
+NoConn ~ 7100 1400
 $EndSCHEMATC
