File: hw/main_logic_board/main_logic_board.kicad_pcb (KiCad board)
At the start: 4 copper layers, 61.9 x 69 mm, 111 parts, among them J1 BATT_IN, J11 SPI1, J12 UART0, J13 UART2, J14 UART4, J15 I2C1, J16 I2C2, J17 5V, J18 3V3, J19 BATT_V, J2 5V_PWR_SEL, J3 3V3_PWR_SEL, J4 USB_A, J5 RC_OUT_1, J6 RC_OUT_2, J7 RC_OUT_3, J8 RC_OUT_4, SW1 ESP_RESET, SW2 ESP_GPIO0, U1 PocketBeagle, U10 ICM-20948, U11 VL53L1X, U12 ACS725xLCTR-40AB, U2 74LVC2T45DC, U3 BME280, U4 NCP1117-5.0_SOT223, U5 NCP1117-3.3_SOT223, U6 TPS563200, U7 TPS563200, U8 ESP-12F, U9 USBLC6-2P6

Commit message: Layout tweaks to power plane
Routing:
- net /telemetry/GPIO15: track 4.25 -> 7.61 mm
- net /RC_OUT_3: track 84.4 -> 85.7 mm
Changed lines of the file:
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@@
     (thickness 1.6)
     (drawings 50)
-    (tracks 1386)
+    (tracks 1400)
     (zones 0)
     (modules 111)
@@
   )
   (setup
-    (last_trace_width 1)
+    (last_trace_width 0.25)
     (user_trace_width 0.2)
     (user_trace_width 0.5)
@@
   (segment (start 134.495685 120.45) (end 141.29 120.45) (width 0.25) (layer B.Cu) (net 28))
   (segment (start 141.29 120.45) (end 141.514999 120.674999) (width 0.25) (layer B.Cu) (net 28))
-  (segment (start 144.730998 121) (end 153.66 121) (width 0.25) (layer B.Cu) (net 28))
-  (segment (start 153.66 121) (end 154.14 120.52) (width 0.25) (layer B.Cu) (net 28))
   (segment (start 166.32 85.799002) (end 167.039002 85.08) (width 0.25) (layer F.Cu) (net 28))
   (segment (start 167.039002 85.08) (end 167.63 85.08) (width 0.25) (layer F.Cu) (net 28))
@@
   (segment (start 165.88 108.35) (end 165.8 108.43) (width 0.25) (layer F.Cu) (net 28))
   (segment (start 165.8 108.43) (end 165.8 108.61) (width 0.25) (layer F.Cu) (net 28))
-  (via (at 154.15 120.51) (size 0.8) (drill 0.4) (layers F.Cu B.Cu) (net 28))
-  (segment (start 154.14 120.52) (end 154.15 120.51) (width 0.25) (layer B.Cu) (net 28))
   (segment (start 159.829002 120.51) (end 160.79 119.549002) (width 0.25) (layer F.Cu) (net 28))
-  (segment (start 154.15 120.51) (end 159.829002 120.51) (width 0.25) (layer F.Cu) (net 28))
   (segment (start 160.79 119.549002) (end 160.79 118.53) (width 0.25) (layer F.Cu) (net 28))
   (segment (start 160.79 118.53) (end 161.31 118.01) (width 0.25) (layer F.Cu) (net 28))
@@
   (segment (start 166.01 86.48) (end 166 86.49) (width 0.25) (layer F.Cu) (net 28))
   (via (at 166.01 86.48) (size 0.8) (drill 0.4) (layers F.Cu B.Cu) (net 28))
+  (segment (start 144.730999 121.000001) (end 145.869999 121.000001) (width 0.25) (layer B.Cu) (net 28))
+  (segment (start 144.730998 121) (end 144.730999 121.000001) (width 0.25) (layer B.Cu) (net 28))
+  (via (at 149.24228 119.735965) (size 0.8) (drill 0.4) (layers F.Cu B.Cu) (net 28))
+  (segment (start 149.24228 119.940722) (end 149.24228 119.735965) (width 0.25) (layer B.Cu) (net 28))
+  (segment (start 145.869999 121.000001) (end 148.183001 121.000001) (width 0.25) (layer B.Cu) (net 28))
+  (segment (start 148.183001 121.000001) (end 149.24228 119.940722) (width 0.25) (layer B.Cu) (net 28))
+  (segment (start 149.24228 119.735965) (end 149.642279 119.335966) (width 0.25) (layer F.Cu) (net 28))
+  (segment (start 151.505966 119.335966) (end 153.665368 119.335966) (width 0.25) (layer F.Cu) (net 28))
+  (segment (start 154.06 119.730598) (end 154.06 119.97) (width 0.25) (layer F.Cu) (net 28))
+  (segment (start 154.06 119.97) (end 154.6 120.51) (width 0.25) (layer F.Cu) (net 28))
+  (segment (start 154.6 120.51) (end 159.83 120.51) (width 0.25) (layer F.Cu) (net 28))
+  (segment (start 159.83 120.51) (end 159.91 120.43) (width 0.25) (layer F.Cu) (net 28))
+  (segment (start 153.665368 119.335966) (end 154.06 119.730598) (width 0.25) (layer F.Cu) (net 28))
+  (segment (start 149.642279 119.335966) (end 151.505966 119.335966) (width 0.25) (layer F.Cu) (net 28))
   (segment (start 139.934 114.14) (end 140.274 113.8) (width 0.25) (layer F.Cu) (net 29))
   (segment (start 138.109 114.14) (end 139.934 114.14) (width 0.25) (layer F.Cu) (net 29))
@@
   (segment (start 138.109 119.22) (end 138.109 118.47) (width 0.25) (layer F.Cu) (net 54))
   (segment (start 138.559 118.02) (end 151.59 118.02) (width 0.25) (layer F.Cu) (net 54))
-  (segment (start 151.59 118.02) (end 152.6 119.03) (width 0.25) (layer F.Cu) (net 54))
-  (segment (start 152.6 119.03) (end 155.88 119.03) (width 0.25) (layer F.Cu) (net 54))
-  (segment (start 155.88 119.03) (end 156.95 117.96) (width 0.25) (layer F.Cu) (net 54))
   (segment (start 156.95 117.96) (end 160.02 117.96) (width 0.25) (layer F.Cu) (net 54))
   (via (at 160.95 117.03) (size 0.8) (drill 0.4) (layers F.Cu B.Cu) (net 54))
@@
   (segment (start 159.73 74) (end 162.15 71.58) (width 0.25) (layer B.Cu) (net 54))
   (segment (start 162.15 71.58) (end 162.15 70.7) (width 0.25) (layer B.Cu) (net 54))
+  (segment (start 156.459002 117.96) (end 155.614001 118.805001) (width 0.25) (layer F.Cu) (net 54))
+  (segment (start 156.95 117.96) (end 156.459002 117.96) (width 0.25) (layer F.Cu) (net 54))
+  (segment (start 154.725999 118.805001) (end 154.244999 118.324001) (width 0.25) (layer F.Cu) (net 54))
+  (segment (start 155.614001 118.805001) (end 154.725999 118.805001) (width 0.25) (layer F.Cu) (net 54))
+  (segment (start 151.59 118.02) (end 153.94 118.02) (width 0.25) (layer F.Cu) (net 54))
+  (segment (start 153.94 118.02) (end 154.26 118.34) (width 0.25) (layer F.Cu) (net 54))
   (segment (start 160.19 77.59) (end 161.12 78.52) (width 0.25) (layer F.Cu) (net 55))
   (segment (start 161.12 78.52) (end 161.12 82.21) (width 0.25) (layer F.Cu) (net 55))
@@
   (segment (start 153.85 124.55) (end 154.825 124.55) (width 0.25) (layer B.Cu) (net 115))
   (segment (start 154.825 124.55) (end 155.8 123.575) (width 0.25) (layer B.Cu) (net 115))
-  (via (at 153.725 122) (size 0.8) (drill 0.4) (layers F.Cu B.Cu) (net 116))
   (segment (start 152.5016 123.317) (end 152.5016 123.2234) (width 0.25) (layer F.Cu) (net 116))
-  (segment (start 152.5016 123.2234) (end 153.725 122) (width 0.25) (layer F.Cu) (net 116))
-  (segment (start 154.290685 122) (end 154.715685 121.575) (width 0.25) (layer B.Cu) (net 116))
-  (segment (start 153.725 122) (end 154.290685 122) (width 0.25) (layer B.Cu) (net 116))
   (segment (start 154.715685 121.575) (end 155.975 121.575) (width 0.25) (layer B.Cu) (net 116))
   (segment (start 141 126.8) (end 139.225 126.8) (width 0.25) (layer F.Cu) (net 117))
@@
   (segment (start 139.43 68.31) (end 138.8 67.68) (width 0.25) (layer B.Cu) (net 107))
   (segment (start 138.8 67.68) (end 137.49 67.68) (width 0.25) (layer B.Cu) (net 107))
+  (via (at 151.599524 121.830913) (size 0.8) (drill 0.4) (layers F.Cu B.Cu) (net 116))
+  (segment (start 152.5016 123.317) (end 152.5016 122.732989) (width 0.25) (layer F.Cu) (net 116))
+  (segment (start 152.5016 122.732989) (end 151.599524 121.830913) (width 0.25) (layer F.Cu) (net 116))
+  (segment (start 152.165209 121.830913) (end 152.436122 121.56) (width 0.25) (layer B.Cu) (net 116))
+  (segment (start 151.599524 121.830913) (end 152.165209 121.830913) (width 0.25) (layer B.Cu) (net 116))
+  (segment (start 152.436122 121.56) (end 155.88 121.56) (width 0.25) (layer B.Cu) (net 116))
   (segment (start 165.894 98.34) (end 165.894 97.756) (width 0.25) (layer F.Cu) (net 130))
   (segment (start 165.894 97.756) (end 165.97 97.68) (width 0.25) (layer F.Cu) (net 130))
@@
     (polygon
       (pts
-        (xy 140.19 78.63) (xy 135.54 80.4) (xy 135.88 83.48) (xy 135.61 114.42) (xy 136.97 116.47)
-        (xy 139.09 117.9) (xy 157.61125 117.775063) (xy 161.16 114.01) (xy 160.88 83.2) (xy 156.38 78.49)
+        (xy 140.275 85.16) (xy 135.69 86.26) (xy 135.72 93.9) (xy 135.61 114.42) (xy 136.97 116.47)
+        (xy 139.09 117.9) (xy 157.61125 117.775063) (xy 161.16 114.01) (xy 160.89 86.29) (xy 156.465 85.02)
       )
     )
