File: hw/main_logic_board/main_logic_board.kicad_pcb (KiCad board)
At the start: 4 copper layers, 61.9 x 69 mm, 111 parts, among them J1 BATT_IN, J11 SPI1, J12 UART0, J13 UART2, J14 UART4, J15 I2C1, J16 I2C2, J17 5V, J18 3V3, J19 BATT_V, J2 5V_PWR_SEL, J3 3V3_PWR_SEL, J4 USB_A, J5 RC_OUT_1, J6 RC_OUT_2, J7 RC_OUT_3, J8 RC_OUT_4, SW1 ESP_RESET, SW2 ESP_GPIO0, U1 PocketBeagle, U10 ICM-20948, U11 VL53L1X, U12 ACS725xLCTR-40AB, U2 74LVC2T45DC, U3 BME280, U4 NCP1117-5.0_SOT223, U5 NCP1117-3.3_SOT223, U6 TPS563200, U7 TPS563200, U8 ESP-12F, U9 USBLC6-2P6

Commit message: Add more silk, + I2C pull ups
Parts:
- added R23: 10K, Resistor_SMD:R_0805_2012Metric, B.Cu at (143.9, 80.4)
- added R24: 10K, Resistor_SMD:R_0805_2012Metric, B.Cu at (143.9, 87.3)
- added R25: 10K, Resistor_SMD:R_0805_2012Metric, B.Cu at (154.8, 86.5)
- added R26: 10K, Resistor_SMD:R_0805_2012Metric, B.Cu at (152.4, 89.3)
- moved J5 5.15 mm to (132.8, 75.2), turned to 90 degrees
- moved C2 0.68 mm to (130.9, 82.7)
- moved C16 0.16 mm to (165.5, 108.7)
- moved C18 0.16 mm to (163.3, 108.7)
- moved C19 0.16 mm to (161.0, 108.7)
Routing:
- net +3V3: track 164.4 -> 180.7 mm, vias 17 -> 19
- net Net-(C21-Pad1): track 14.5 -> 9.10 mm, vias 2 -> 0
- net /I2C2_SCL: track 53.2 -> 58.2 mm
- net /I2C1_SDA: track 43.3 -> 47.6 mm
- net /I2C1_SCL: track 36.5 -> 40.8 mm
- net /I2C2_SDA: track 52.4 -> 56.4 mm, vias 2 -> 3
- net +5V: track 234.6 -> 236.8 mm
- net /UART4_TX: track 75.3 -> 74.7 mm
Other:
- board text added: "3V3"
- board text added: "5V"
- board text added: "BATT"
- board text added: "GND"
- board text added: "GND|"
- board text added: "LDO"
- board text added: "RCO_1"
- board text added: "RCO_2"
- board text added: "RCO_3"
- board text added: "RCO_4"
- board text added: "RX"
- board text added: "SCL"
- board text added: "SDA"
- board text added: "SW"
- board text added: "TX"
