File: hw/main_logic_board/actuation.sch (KiCad schematic (older format))
At the start: 6 parts, among them U2 74LVC2T45DC

Commit message: Add 3D model files, lay out switching circuit, other tweaks
Parts:
- BZ1: footprint (none) -> Buzzer_Beeper:Buzzer_Murata_PKMCS0909E4000-R1
Connections:
- net BUZZER_PWM: now also BZ1.1 (-)
- net GND: now also BZ1.2 (+)
Other:
- moved on the sheet: BZ1
Changed lines of the file:
@@
 L Device:Buzzer BZ1
 U 1 1 5EB6C9F9
-P 4650 3850
-F 0 "BZ1" H 4802 3879 50  0000 L CNN
-F 1 "Buzzer" H 4802 3788 50  0000 L CNN
-F 2 "" V 4625 3950 50  0001 C CNN
-F 3 "~" V 4625 3950 50  0001 C CNN
-	1    4650 3850
+P 2750 3450
+F 0 "BZ1" H 2902 3479 50  0000 L CNN
+F 1 "Buzzer" H 2902 3388 50  0000 L CNN
+F 2 "Buzzer_Beeper:Buzzer_Murata_PKMCS0909E4000-R1" V 2725 3550 50  0001 C CNN
+F 3 "~" V 2725 3550 50  0001 C CNN
+	1    2750 3450
 	1    0    0    -1
 $EndComp
@@
 Text HLabel 8050 1950 2    50   Input ~ 0
 LED_DATA_OUT
-Text HLabel 3600 3750 0    50   Input ~ 0
+Text HLabel 1700 3350 0    50   Input ~ 0
 BUZZER_PWM
+Wire Wire Line
+	2650 3350 1700 3350
+Wire Wire Line
+	2650 3550 2600 3550
+Wire Wire Line
+	2600 3550 2600 3900
+$Comp
+L power:GND #PWR0135
+U 1 1 5ECA99DD
+P 2600 3900
+F 0 "#PWR0135" H 2600 3650 50  0001 C CNN
+F 1 "GND" H 2605 3727 50  0000 C CNN
+F 2 "" H 2600 3900 50  0001 C CNN
+F 3 "" H 2600 3900 50  0001 C CNN
+	1    2600 3900
+	1    0    0    -1
+$EndComp
 $EndSCHEMATC

Commit message: Adding BOM information
Parts:
- BZ1: Digikey (none) -> https://www.digikey.ca/product-detail/en/pui-audio-inc/SMT-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
- D1, D2, D3, D4: Digikey (none) -> N/A
Changed lines of the file:
@@
 F 2 "LED_SMD:LED_WS2812_PLCC6_5.0x5.0mm_P1.6mm" H 3900 1650 50  0001 L TNN
 F 3 "http://www.normandled.com/upload/201605/WS2813%20LED%20Datasheet.pdf" H 3950 1575 50  0001 L TNN
+F 4 "N/A" H 3850 1950 50  0001 C CNN "Digikey"
 	1    3850 1950
 	1    0    0    -1
@@
 F 2 "LED_SMD:LED_WS2812_PLCC6_5.0x5.0mm_P1.6mm" H 6150 1650 50  0001 L TNN
 F 3 "http://www.normandled.com/upload/201605/WS2813%20LED%20Datasheet.pdf" H 6200 1575 50  0001 L TNN
+F 4 "N/A" H 6100 1950 50  0001 C CNN "Digikey"
 	1    6100 1950
 	1    0    0    -1
@@
 F 2 "LED_SMD:LED_WS2812_PLCC6_5.0x5.0mm_P1.6mm" H 5050 1650 50  0001 L TNN
 F 3 "http://www.normandled.com/upload/201605/WS2813%20LED%20Datasheet.pdf" H 5100 1575 50  0001 L TNN
+F 4 "N/A" H 5000 1950 50  0001 C CNN "Digikey"
 	1    5000 1950
 	1    0    0    -1
@@
 F 2 "LED_SMD:LED_WS2812_PLCC6_5.0x5.0mm_P1.6mm" H 7200 1650 50  0001 L TNN
 F 3 "http://www.normandled.com/upload/201605/WS2813%20LED%20Datasheet.pdf" H 7250 1575 50  0001 L TNN
+F 4 "N/A" H 7150 1950 50  0001 C CNN "Digikey"
 	1    7150 1950
 	1    0    0    -1
@@
 F 1 "Buzzer" H 2902 3388 50  0000 L CNN
 F 2 "Buzzer_Beeper:Buzzer_Murata_PKMCS0909E4000-R1" V 2725 3550 50  0001 C CNN
-F 3 "~" V 2725 3550 50  0001 C CNN
+F 3 "http://www.puiaudio.com/pdf/SMT-0927-S-7-R.pdf" V 2725 3550 50  0001 C CNN
+F 4 "https://www.digikey.ca/product-detail/en/pui-audio-inc/SMT-0927-S-7-R/668-1664-1-ND/9083419" H 2750 3450 50  0001 C CNN "Digikey"
 	1    2750 3450
 	1    0    0    -1

Commit message: Update repo with latest local
Parts:
- D1, D2, D3, D4: Digikey N/A -> (none)
- U2: Digikey (none) -> https://www.digikey.ca/product-detail/en/nexperia-usa-inc/7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
Changed lines of the file:
@@
 F 2 "LED_SMD:LED_WS2812_PLCC6_5.0x5.0mm_P1.6mm" H 3900 1650 50  0001 L TNN
 F 3 "http://www.normandled.com/upload/201605/WS2813%20LED%20Datasheet.pdf" H 3950 1575 50  0001 L TNN
-F 4 "N/A" H 3850 1950 50  0001 C CNN "Digikey"
+F 4 "" H 3850 1950 50  0001 C CNN "Digikey"
 	1    3850 1950
 	1    0    0    -1
@@
 F 2 "LED_SMD:LED_WS2812_PLCC6_5.0x5.0mm_P1.6mm" H 6150 1650 50  0001 L TNN
 F 3 "http://www.normandled.com/upload/201605/WS2813%20LED%20Datasheet.pdf" H 6200 1575 50  0001 L TNN
-F 4 "N/A" H 6100 1950 50  0001 C CNN "Digikey"
+F 4 "" H 6100 1950 50  0001 C CNN "Digikey"
 	1    6100 1950
 	1    0    0    -1
@@
 F 2 "LED_SMD:LED_WS2812_PLCC6_5.0x5.0mm_P1.6mm" H 5050 1650 50  0001 L TNN
 F 3 "http://www.normandled.com/upload/201605/WS2813%20LED%20Datasheet.pdf" H 5100 1575 50  0001 L TNN
-F 4 "N/A" H 5000 1950 50  0001 C CNN "Digikey"
+F 4 "" H 5000 1950 50  0001 C CNN "Digikey"
 	1    5000 1950
 	1    0    0    -1
@@
 F 2 "LED_SMD:LED_WS2812_PLCC6_5.0x5.0mm_P1.6mm" H 7200 1650 50  0001 L TNN
 F 3 "http://www.normandled.com/upload/201605/WS2813%20LED%20Datasheet.pdf" H 7250 1575 50  0001 L TNN
-F 4 "N/A" H 7150 1950 50  0001 C CNN "Digikey"
+F 4 "" H 7150 1950 50  0001 C CNN "Digikey"
 	1    7150 1950
 	1    0    0    -1
@@
 F 2 "Package_SO:VSSOP-8_2.3x2mm_P0.5mm" H 2050 1200 50  0001 C CNN
 F 3 "https://assets.nexperia.com/documents/data-sheet/74LVC_LVCH2T45.pdf" H 2300 1800 50  0001 C CNN
+F 4 "https://www.digikey.ca/product-detail/en/nexperia-usa-inc/74LVC2T45DC-125/1727-4578-1-ND/2530957" H 2050 2050 50  0001 C CNN "Digikey"
 	1    2050 2050
 	1    0    0    -1
