File: hw/main_logic_board/sensors.sch (KiCad schematic (older format))
At the start: 5 parts, among them U2 MPU-9250, U3 BME280

Commit message: Finish initial power schematics, swap some footprints for visualization in pcb view
Parts:
- gave numbers to parts that had none: 3
Changed lines of the file:
@@
 $EndComp
 $Comp
-L power:+3V3 #PWR?
+L power:+3V3 #PWR0108
 U 1 1 5EA7141D
 P 3000 1300
-F 0 "#PWR?" H 3000 1150 50  0001 C CNN
+F 0 "#PWR0108" H 3000 1150 50  0001 C CNN
 F 1 "+3V3" H 3015 1473 50  0000 C CNN
 F 2 "" H 3000 1300 50  0001 C CNN
@@
 $EndComp
 $Comp
-L power:+3V3 #PWR?
+L power:+3V3 #PWR0109
 U 1 1 5EA72BD4
 P 3050 4500
-F 0 "#PWR?" H 3050 4350 50  0001 C CNN
+F 0 "#PWR0109" H 3050 4350 50  0001 C CNN
 F 1 "+3V3" H 3065 4673 50  0000 C CNN
 F 2 "" H 3050 4500 50  0001 C CNN
@@
 AR Path="/5E9DC864/5EA73DF2" Ref="C?"  Part="1"
 AR Path="/5EA73DF2" Ref="C?"  Part="1"
-AR Path="/5E9DC684/5EA73DF2" Ref="C?"  Part="1"
-F 0 "C?" H 2458 4796 50  0000 R CNN
+AR Path="/5E9DC684/5EA73DF2" Ref="C5"  Part="1"
+F 0 "C5" H 2458 4796 50  0000 R CNN
 F 1 "100nF" H 2458 4705 50  0000 R CNN
 F 2 "" H 2550 4750 50  0001 C CNN
@@
 $EndComp
 $Comp
-L power:GND #PWR?
+L power:GND #PWR0110
 U 1 1 5EA7446C
 P 2550 4950
-F 0 "#PWR?" H 2550 4700 50  0001 C CNN
+F 0 "#PWR0110" H 2550 4700 50  0001 C CNN
 F 1 "GND" H 2555 4777 50  0000 C CNN
 F 2 "" H 2550 4950 50  0001 C CNN
@@
 AR Path="/5E9DC864/5EA73A6B" Ref="C?"  Part="1"
 AR Path="/5EA73A6B" Ref="C?"  Part="1"
-AR Path="/5E9DC684/5EA73A6B" Ref="C?"  Part="1"
-F 0 "C?" H 2158 1596 50  0000 R CNN
+AR Path="/5E9DC684/5EA73A6B" Ref="C4"  Part="1"
+F 0 "C4" H 2158 1596 50  0000 R CNN
 F 1 "100nF" H 2158 1505 50  0000 R CNN
 F 2 "" H 2250 1550 50  0001 C CNN
@@
 	2550 4850 2550 4950
 $Comp
-L power:GND #PWR?
+L power:GND #PWR0111
 U 1 1 5EA77C58
 P 2250 1700
-F 0 "#PWR?" H 2250 1450 50  0001 C CNN
+F 0 "#PWR0111" H 2250 1450 50  0001 C CNN
 F 1 "GND" H 2255 1527 50  0000 C CNN
 F 2 "" H 2250 1700 50  0001 C CNN
@@
 NoConn ~ 3800 2250
 $Comp
-L power:GND #PWR?
+L power:GND #PWR0112
 U 1 1 5EA78CFF
 P 3100 3550
-F 0 "#PWR?" H 3100 3300 50  0001 C CNN
+F 0 "#PWR0112" H 3100 3300 50  0001 C CNN
 F 1 "GND" H 3105 3377 50  0000 C CNN
 F 2 "" H 3100 3550 50  0001 C CNN
@@
 	3100 3550 3100 3450
 $Comp
-L power:GND #PWR?
+L power:GND #PWR0113
 U 1 1 5EA79BF7
 P 3050 6100
-F 0 "#PWR?" H 3050 5850 50  0001 C CNN
+F 0 "#PWR0113" H 3050 5850 50  0001 C CNN
 F 1 "GND" H 3055 5927 50  0000 C CNN
 F 2 "" H 3050 6100 50  0001 C CNN
@@
 AR Path="/5E9DC864/5EA7B1AC" Ref="C?"  Part="1"
 AR Path="/5EA7B1AC" Ref="C?"  Part="1"
-AR Path="/5E9DC684/5EA7B1AC" Ref="C?"  Part="1"
-F 0 "C?" V 4529 2750 50  0000 C CNN
+AR Path="/5E9DC684/5EA7B1AC" Ref="C6"  Part="1"
+F 0 "C6" V 4529 2750 50  0000 C CNN
 F 1 "100nF" V 4438 2750 50  0000 C CNN
 F 2 "" H 4300 2750 50  0001 C CNN
@@
 	4200 2750 3800 2750
 $Comp
-L power:GND #PWR?
+L power:GND #PWR0114
 U 1 1 5EA7BBE7
 P 4450 2750
-F 0 "#PWR?" H 4450 2500 50  0001 C CNN
+F 0 "#PWR0114" H 4450 2500 50  0001 C CNN
 F 1 "GND" H 4455 2577 50  0000 C CNN
 F 2 "" H 4450 2750 50  0001 C CNN
@@
 	4400 2750 4450 2750
 $Comp
-L power:+3V3 #PWR?
+L power:+3V3 #PWR0115
 U 1 1 5EA7FF97
 P 4000 2650
-F 0 "#PWR?" H 4000 2500 50  0001 C CNN
+F 0 "#PWR0115" H 4000 2500 50  0001 C CNN
 F 1 "+3V3" H 4015 2823 50  0000 C CNN
 F 2 "" H 4000 2650 50  0001 C CNN
@@
 	4000 2850 4000 2650
 $Comp
-L power:GND #PWR?
+L power:GND #PWR0116
 U 1 1 5EA80B48
 P 4000 3000
-F 0 "#PWR?" H 4000 2750 50  0001 C CNN
+F 0 "#PWR0116" H 4000 2750 50  0001 C CNN
 F 1 "GND" H 4005 2827 50  0000 C CNN
 F 2 "" H 4000 3000 50  0001 C CNN
@@
 MPU_CS
 $Comp
-L power:GND #PWR?
+L power:GND #PWR0117
 U 1 1 5EA833A5
 P 2300 2900
-F 0 "#PWR?" H 2300 2650 50  0001 C CNN
+F 0 "#PWR0117" H 2300 2650 50  0001 C CNN
 F 1 "GND" H 2305 2727 50  0000 C CNN
 F 2 "" H 2300 2900 50  0001 C CNN

Commit message: Finish prelim schematic + PCB component placement
Parts:
- added C20, C21, C22: 100n, Capacitor_SMD:C_0805_2012Metric, symbol Device:C_Small
- added U10: ICM-20948, Sensor_Motion:InvenSense_QFN-24_3x3mm_P0.4mm, symbol Sensor_Motion:ICM-20948
- added U11: VL53L1X, Sensor_Distance:ST_VL53L1x, symbol VL53L1Xlib:VL53L1X
- C4, C5, C6: value 100nF -> 100n; footprint (none) -> Capacitor_SMD:C_0805_2012Metric
Connections:
- net labels added: BME_CS_N, ICM_CS_N, ICM_MISO, ICM_MOSI_SDA, ICM_SCLK_SCL, MPU_CS_N, VL_SCL, VL_SDA
- net labels removed: BME_CS, MPU_CS
- wire segments 37 -> 74
- no-connect marks 3 -> 8
Other:
- moved on the sheet: C4, C5, C6, U3

Commit message: Add debug headers, LED wiring, remove MPU
Parts:
- removed C4, C6: 100n, Capacitor_SMD:C_0805_2012Metric, symbol Device:C_Small
- removed U2: MPU-9250, Sensor_Motion:InvenSense_QFN-24_3x3mm_P0.4mm, symbol Sensor_Motion:MPU-9250
Connections:
- net labels removed: MPU_CS_N, MPU_MISO, MPU_MOSI_SDA, MPU_SCLK_SCL
- wire segments 74 -> 53
- no-connect marks 8 -> 5
Other:
- moved on the sheet: C20, C21, C22, U10, U11

Commit message: Update repo with latest local
Parts:
- U10: Digikey (none) -> https://www.digikey.ca/product-detail/en/tdk-invensense/ICM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
- U11: Digikey (none) -> https://www.digikey.ca/product-detail/en/stmicroelectronics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
- U3: Digikey (none) -> https://www.digikey.ca/product-detail/en/bosch-sensortec/BM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
Changed lines of the file:
@@
 F 2 "Package_LGA:Bosch_LGA-8_2.5x2.5mm_P0.65mm_ClockwisePinNumbering" H 4350 5350 50  0001 C CNN
 F 3 "https://ae-bst.resource.bosch.com/media/_tech/media/datasheets/BST-BME280-DS002.pdf" H 2850 5600 50  0001 C CNN
+F 4 "https://www.digikey.ca/product-detail/en/bosch-sensortec/BME280/828-1063-1-ND/6136314" H 2850 5800 50  0001 C CNN "Digikey"
 	1    2850 5800
 	1    0    0    -1
@@
 F 2 "Sensor_Motion:InvenSense_QFN-24_3x3mm_P0.4mm" H 3350 1500 50  0001 C CNN
 F 3 "http://www.invensense.com/wp-content/uploads/2016/06/DS-000189-ICM-20948-v1.3.pdf" H 3350 2350 50  0001 C CNN
+F 4 "https://www.digikey.ca/product-detail/en/tdk-invensense/ICM-20948/1428-1123-1-ND/7062698" H 3350 2500 50  0001 C CNN "Digikey"
 	1    3350 2500
 	1    0    0    -1
@@
 F 2 "Sensor_Distance:ST_VL53L1x" H 7850 2050 50  0001 C CNN
 F 3 "https://www.st.com/resource/en/datasheet/vl53l1x.pdf" H 7850 2050 50  0001 C CNN
+F 4 "https://www.digikey.ca/product-detail/en/stmicroelectronics/VL53L1CXV0FY-1/497-17764-1-ND/8276742" H 7800 2000 50  0001 C CNN "Digikey"
 	1    7800 2000
 	1    0    0    -1
